Commit message: Added camera to robot xacro

File: src/my_robot/urdf/my_robot.xacro (robot description, xacro)
@@ -117,3 +117,32 @@
     </visual>
   </link>
+  <joint name="camera_joint" type="fixed">
+    <origin xyz="0 0 0" rpy="0 0 0" />
+    <axis xyz="0 1 0" rpy="0 0 0"/>
+    <parent link="chassis"/>
+    <child link="camera" />
+  </joint>
+  <link name='camera'>
+    <inertial>
+        <mass value="0.1"/>
+        <origin xyz="0.2 0 0" rpy=" 0 0 0"/>
+        <inertia
+            ixx="1e-6" ixy="0" ixz="0"
+            iyy="1e-6" iyz="0"
+            izz="1e-6"
+        />
+    </inertial>
+    <collision name='camera_collision'>
+      <origin xyz="0.2 0 0" rpy=" 0 0 0"/>
+      <geometry>
+        <box size=".05 .05 .05"/>
+      </geometry>
+    </collision>
+    <visual name='camera_visual'>
+      <origin xyz="0.2 0 0" rpy=" 0 0 0"/>
+      <geometry>
+       <box size=".05 .05 .05"/>
+      </geometry>
+    </visual>
+  </link>
 </robot>

Commit message: Added lidar

File: src/my_robot/urdf/my_robot.xacro (robot description, xacro)
@@ -146,3 +146,44 @@
     </visual>
   </link>
+  <joint name="hokuyo_joint" type="fixed">
+    <origin xyz="0.15 0 0.1" rpy="0 0 0" />
+    <axis xyz="0 1 0" rpy="0 0 0"/>
+    <parent link="chassis"/>
+    <child link="hokuyo" />
+  </joint>
+  <link name='hokuyo'>
+    <inertial>
+        <mass value="1e-5"/>
+        <origin xyz="0 0 0" rpy=" 0 0 0"/>
+        <inertia
+            ixx="1e-6" ixy="0" ixz="0"
+            iyy="1e-6" iyz="0"
+            izz="1e-6"
+        />
+    </inertial>
+    <collision name='hokuyo_collision'>
+      <origin xyz="0 0 0" rpy=" 0 0 0"/>
+      <geometry>
+        <box size=".1 .1 .1"/>
+      </geometry>
+    </collision>
+    <visual name='hokuyo_visual'>
+      <origin xyz="0 0 0" rpy=" 0 0 0"/>
+      <geometry>
+       <mesh filename="package://my_robot/meshes/hokuyo.dae"/>
+      </geometry>
+    </visual>
+  </link>
+  <gazebo reference="left_wheel">
+    <material>Gazebo/Yellow</material>
+  </gazebo>
+  <gazebo reference="right_wheel">
+    <material>Gazebo/Yellow</material>
+  </gazebo>
+  <gazebo reference="chassis">
+    <material>Gazebo/Blue</material>
+  </gazebo>
+  <gazebo reference="camera">
+    <material>Gazebo/Red</material>
+  </gazebo>
 </robot>

Commit message: adjust camera location

File: src/my_robot/urdf/my_robot.xacro (robot description, xacro)
@@ -119,5 +119,5 @@
   </link>
   <joint name="camera_joint" type="fixed">
-    <origin xyz="0 0 0" rpy="0 0 0" />
+    <origin xyz="0.2 0 0" rpy="0 0 0" />
     <axis xyz="0 1 0" rpy="0 0 0"/>
     <parent link="chassis"/>
@@ -127,5 +127,5 @@
     <inertial>
         <mass value="0.1"/>
-        <origin xyz="0.2 0 0" rpy=" 0 0 0"/>
+        <origin xyz="0 0 0" rpy=" 0 0 0"/>
         <inertia
             ixx="1e-6" ixy="0" ixz="0"
@@ -135,5 +135,5 @@
     </inertial>
     <collision name='camera_collision'>
-      <origin xyz="0.2 0 0" rpy=" 0 0 0"/>
+      <origin xyz="0 0 0" rpy=" 0 0 0"/>
       <geometry>
         <box size=".05 .05 .05"/>
@@ -141,5 +141,5 @@
     </collision>
     <visual name='camera_visual'>
-      <origin xyz="0.2 0 0" rpy=" 0 0 0"/>
+      <origin xyz="0 0 0" rpy=" 0 0 0"/>
       <geometry>
        <box size=".05 .05 .05"/>
